Commit message: Add robot description links and meshes for SKD-100 sensors

File: skd100_description/urdf/core.urdf.xacro (robot description, xacro)
@@ -100,3 +100,127 @@
 		left_side="false"
 		/>
+	<!-- Sensors -->
+	<!-- Z-coordinate of the sensor deck relative to base_link -->
+	<xacro:property name="sensor_base_z_coord" value="0.130" />
+	<!-- Base deck for sensors -->
+    <link name="base_sensors">
+		<xacro:dummy_inertial />
+	</link>
+    <joint name="base_sensors_joint" type="fixed">
+        <origin xyz="0 0 ${sensor_base_z_coord+chassis_z_coord}" rpy="0 0 0" />
+        <parent link="base_link" />
+        <child link="base_sensors" />
+    </joint>
+	<!-- MTI630 IMU -->
+	<link name="xsens_imu_link">
+		<visual>
+			<origin xyz="0 0 ${-0.025/2}" rpy="0 0 0"/>
+			<geometry>
+				<box size="0.065 0.050 0.025"/>
+			</geometry>
+			<material name="Pink">
+				<color rgba="${255/255} ${0/255} ${255/255} 1.0"/>
+			</material>
+		</visual>
+		<xacro:dummy_inertial />
+	</link>
+	<joint name="xsens_imu_joint" type="fixed">
+		<parent link="base_link" />
+		<child link="xsens_imu_link" />
+		<origin xyz="0 0 ${chassis_z_size/2 + 0.135}" rpy="0 0 0" />
+	</joint>
+	<!-- RPLidar S3 -->
+	<link name="rplidar_link">
+		<xacro:dummy_inertial />
+		<collision>
+			<origin xyz="0 0 ${0.0413/2}" rpy="0 0 0"/>
+			<geometry>
+				<!-- 59.80 mm x 55.60 mm x 41.30 mm -->
+				<box size="${0.05980} ${0.05560} ${0.0413}"/>
+			</geometry>
+		</collision>
+		<visual>
+			<origin xyz="0 0 ${0.0135}" rpy="${pi/2} 0 ${-pi/2}"/>
+			<geometry>
+				<mesh filename="package://skd100_description/meshes/rplidar_s3.stl"  scale="0.001 0.001 0.001"/>
+			</geometry>
+			<material name="Green">
+				<color rgba="${0/255} ${255/255} ${0/255} 1.0"/>
+			</material>
+		</visual>
+	</link>
+	<joint name="rplidar_joint" type="fixed">
+		<parent link="base_sensors"/>
+		<child link="rplidar_link"/>
+		<!-- Base: 5mm up and 103.2mm to front -->
+		<origin xyz="${0.1032} 0 ${0.005}" rpy="0 0 0"/>
+	</joint>
+	<link name="rplidar_optical_link">
+		<xacro:dummy_inertial />
+	</link>
+	<!-- Optical window: 29.8mm up  -->
+	<!-- The RPLIDAR S3 adopts a coordinate system of the left hand -->
+    <joint name="rplidar_optical_joint" type="fixed">
+        <origin xyz="0 0 ${0.0298}" rpy="0 0 ${pi}" />
+        <parent link="rplidar_link" />
+        <child link="rplidar_optical_link" />
+    </joint>
+	<!-- Bridge for GPS antenna -->
+	<!-- Z-coordinate of the antenna base relative to base_link -->
+	<xacro:property name="antenna_base_z_coord" value="0.4" />
+    <link name="antenna_base">
+		<visual>
+			<origin xyz="0 0 0" rpy="0 0 0"/>
+			<geometry>
+				<box size="${0.04} ${1.2} ${0.02}"/>
+			</geometry>
+			<material name="White">
+				<color rgba="${255/255} ${255/255} ${255/255} 1.0"/>
+			</material>
+		</visual>
+		<xacro:dummy_inertial />
+	</link>
+    <joint name="antenna_base_joint" type="fixed">
+        <origin xyz="0 0 ${antenna_base_z_coord+chassis_z_coord}" rpy="0 0 0" />
+        <parent link="base_link" />
+        <child link="antenna_base" />
+    </joint>
+	<!-- Z-coordinate of the antenna base relative to base_link -->
+	<xacro:property name="gps_antenna_separation" value="1.0" />
+	<!-- Ardusimple RTK Heading rover antenna -->
+	<link name="gps_main_antenna_link">
+		<visual>
+			<origin xyz="0 0 ${0.006}" rpy="0 0 0"/>
+			<geometry>
+				<mesh filename="package://skd100_description/meshes/ANT2B-ANN.stl"  scale="0.001 0.001 0.001"/>
+			</geometry>
+			<material name="Yellow">
+				<color rgba="1.0 1.0 0.0 1.0"/>
+			</material>
+		</visual>
+		<xacro:dummy_inertial />
+	</link>
+	<joint name="gps_main_antenna_joint" type="fixed">
+		<parent link="antenna_base" />
+		<child link="gps_main_antenna_link" />
+		<origin xyz="0 ${gps_antenna_separation/2} ${0.01}" rpy="0 0 0" />
+	</joint>
+	<!-- Ardusimple RTK Heading moving base antenna -->
+	<link name="gps_second_antenna_link">
+		<visual>
+			<origin xyz="0 0 ${0.006}" rpy="0 0 ${-pi/2}"/>
+			<geometry>
+				<mesh filename="package://skd100_description/meshes/ANT2B-ANN.stl"  scale="0.001 0.001 0.001"/>
+			</geometry>
+			<material name="Yellow">
+				<color rgba="1.0 1.0 0.0 1.0"/>
+			</material>
+		</visual>
+		<xacro:dummy_inertial />
+	</link>
+	<joint name="gps_second_antenna_joint" type="fixed">
+		<parent link="antenna_base" />
+		<child link="gps_second_antenna_link" />
+		<origin xyz="0 ${-gps_antenna_separation/2} ${0.01}" rpy="0 0 0" />
+	</joint>
 </robot>

Commit message: Fix ANT2B-ANN visual mesh orientation

File: skd100_description/urdf/core.urdf.xacro (robot description, xacro)
@@ -191,5 +191,5 @@
 	<link name="gps_main_antenna_link">
 		<visual>
-			<origin xyz="0 0 ${0.006}" rpy="0 0 0"/>
+			<origin xyz="0 0 ${0.006}" rpy="0 0 ${pi}"/>
 			<geometry>
 				<mesh filename="package://skd100_description/meshes/ANT2B-ANN.stl"  scale="0.001 0.001 0.001"/>
@@ -209,5 +209,5 @@
 	<link name="gps_second_antenna_link">
 		<visual>
-			<origin xyz="0 0 ${0.006}" rpy="0 0 ${-pi/2}"/>
+			<origin xyz="0 0 ${0.006}" rpy="0 0 ${pi}"/>
 			<geometry>
 				<mesh filename="package://skd100_description/meshes/ANT2B-ANN.stl"  scale="0.001 0.001 0.001"/>
